File: PTP_LV1/PTP_LV1.kicad_pcb (KiCad board)
At the start: 2 copper layers, 45 parts, among them U1 LM2574N-5, U2 4027, U3 4027, U4 74LS47, U5 FYS-3911BUHR-21, U6 SN74LVC1G11, U7 NE555P

Commit message: twe
rtzert
Parts:
- moved R19 91.0 mm to (110.5, 103.5), turned to 90 degrees
- moved U6 36.9 mm to (169.5, 81.5)
- moved R17 23.6 mm to (183.6, 89.0)
- moved D5 22.9 mm to (176.5, 74.0)
- moved R4 22.2 mm to (174.4, 69.0), turned to 90 degrees
- moved D1 22.0 mm to (154.0, 74.0)
- moved L1 21.2 mm to (144.5, 77.0), turned to 90 degrees
- moved R1 21.2 mm to (155.0, 68.7), turned to 90 degrees
- moved R9 19.4 mm to (168.0, 117.5), turned to 90 degrees
- moved R15 18.0 mm to (180.0, 117.5), turned to 90 degrees
- moved R6 17.4 mm to (183.6, 98.0)
- moved R12 16.4 mm to (176.0, 117.5), turned to 90 degrees
- moved SW2 15.2 mm to (138.0, 100.6), turned to -90 degrees
- moved R10 13.5 mm to (172.5, 117.5), turned to 90 degrees
- moved R11 13.5 mm to (183.6, 86.0)
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Routing:
- net GND: track 0.00 -> 104.3 mm, vias 0 -> 1
- net Q3: track 0.00 -> 52.6 mm, vias 0 -> 2
- net +5V: track 0.00 -> 51.4 mm
- net Q0: track 0.00 -> 50.2 mm
- net Q1: track 0.00 -> 48.1 mm, vias 0 -> 2
- net Q2: track 0.00 -> 47.7 mm
- net Net-(U3A-J): track 0.00 -> 47.3 mm
- net Net-(D4-K): track 0.00 -> 33.1 mm
- net Net-(U2A-J): track 0.00 -> 33.0 mm
- net VD: track 0.00 -> 27.1 mm
- net Net-(U2B-J): track 0.00 -> 26.4 mm
- net Net-(U5-A): track 0.00 -> 23.4 mm
- net Reset: track 0.00 -> 22.7 mm, vias 0 -> 2
- net Net-(U5-B): track 0.00 -> 22.3 mm
- net Net-(U5-C): track 0.00 -> 21.9 mm
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Other:
- board text added: "H4"

Commit message: Nikpalj LV7
sbe gotovo sad na seminar najjace
Parts:
- U6: footprint Package_TO_SOT_SMD:SOT-23_Handsoldering -> Package_TO_SOT_SMD:SOT-23-6
Routing:
- net +5V: track 51.4 -> 259.6 mm, vias 0 -> 9
- net Clock: track 13.0 -> 74.7 mm, vias 0 -> 4
- net GND: track 104.3 -> 69.6 mm, vias 1 -> 2
- net Net-(U7-THR): track 0.00 -> 27.2 mm, vias 0 -> 2
- net 555: track 0.00 -> 26.8 mm
- net Net-(SW2-A): track 0.00 -> 26.7 mm
- net Reset: track 22.7 -> 44.9 mm, vias 2 -> 5
- net Net-(U7-DIS): track 0.00 -> 19.2 mm
- net Net-(R13-Pad1): track 0.00 -> 16.7 mm
- net VD: track 27.1 -> 35.1 mm
- net Net-(U4-BI): track 21.6 -> 26.7 mm
- net Net-(U5-E): track 19.7 -> 23.9 mm
- net Q3: track 52.6 -> 48.8 mm
- net Net-(U3A-J): track 47.3 -> 49.9 mm
- net Net-(U2A-J): track 33.0 -> 35.5 mm
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- added copper zone on B.Cu, net GND
Other:
- board outline added: 100 x 80 mm
