File: PTP_LV1/PTP_LV1.kicad_sch (KiCad schematic)
At the start: 45 parts, among them U1 LM2574N-5, U2 4027, U3 4027, U4 74LS47, U5 FYS-3911BUHR-21, U6 SN74LVC1G11, U7 NE555P

Commit message: Nikpalj LV7
sbe gotovo sad na seminar najjace
Parts:
- U6: footprint Package_TO_SOT_SMD:SOT-23_Handsoldering -> Package_TO_SOT_SMD:SOT-23-6
Changed lines of the file:
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@@
 			)
 		)
-		(property "Footprint" "Package_TO_SOT_SMD:SOT-23_Handsoldering"
+		(property "Footprint" "Package_TO_SOT_SMD:SOT-23-6"
 			(at 153.67 146.05 0)
 			(effects
